Commit message: First commit

File: robots/defined.urdf.xacro (robot description, xacro)
@@ -2,7 +2,7 @@
 <robot xmlns:xacro="http://www.ros.org/wiki/xacro" name="panda">
   <xacro:include filename="$(find franka_description)/robots/panda_arm_hand.urdf.xacro"/>
+  <xacro:include filename="$(find franka_description)/robots/panda.transmission.xacro" />
   <xacro:include filename="$(find franka_description)/robots/panda.gazebo.xacro" />
-  <xacro:include filename="$(find franka_description)/robots/panda.transmission.xacro" />
+  <xacro:panda_transmission arm_id="panda" />s
   <xacro:panda_gazebo arm_id="panda" />
-  <xacro:panda_transmission arm_id="panda"/>
 </robot>

File: robots/panda.gazebo.xacro (robot description, xacro)
@@ -62,4 +62,9 @@
             <mu2>0.2</mu2>
         </gazebo> -->
+        <gazebo>
+            <plugin name="gazebo_ros_control" filename="libgazebo_ros_control.so">
+                <robotNamespace>/panda</robotNamespace>
+            </plugin>
+        </gazebo>
     </xacro:macro>
 </robot>

File: robots/panda_arm.xacro (robot description, xacro)
@@ -71,5 +71,5 @@
         <origin xyz="0 0 0" rpy="0 0 0" />
         <inertia ixx="0.3" ixy="0.0" ixz="0.0" iyy="0.3" iyz="0.0" izz="0.3" />
-        <mass value="3.06" />
+        <mass value="2.34471" />
       </inertial>
     </link>
@@ -110,5 +110,5 @@
         <origin xyz="0 0 0" rpy="0 0 0" />
         <inertia ixx="0.3" ixy="0.0" ixz="0.0" iyy="0.3" iyz="0.0" izz="0.3" />
-        <mass value="3.06" />
+        <mass value="2.36414" />
       </inertial>
     </link>
@@ -149,5 +149,5 @@
         <origin xyz="0 0 0" rpy="0 0 0" />
         <inertia ixx="0.3" ixy="0.0" ixz="0.0" iyy="0.3" iyz="0.0" izz="0.3" />
-        <mass value="3.06" />
+        <mass value="2.38050" />
       </inertial>
     </link>
@@ -188,5 +188,5 @@
         <origin xyz="0 0 0" rpy="0 0 0" />
         <inertia ixx="0.3" ixy="0.0" ixz="0.0" iyy="0.3" iyz="0.0" izz="0.3" />
-        <mass value="3.06" />
+        <mass value="2.42754" />
       </inertial>
     </link>
@@ -245,5 +245,5 @@
         <origin xyz="0 0 0" rpy="0 0 0" />
         <inertia ixx="0.3" ixy="0.0" ixz="0.0" iyy="0.3" iyz="0.0" izz="0.3" />
-        <mass value="3.06" />
+        <mass value="3.49611" />
       </inertial>
     </link>
@@ -284,5 +284,5 @@
         <origin xyz="0 0 0" rpy="0 0 0" />
         <inertia ixx="0.3" ixy="0.0" ixz="0.0" iyy="0.3" iyz="0.0" izz="0.3" />
-        <mass value="3.06" />
+        <mass value="1.46736" />
       </inertial>
     </link>
@@ -323,5 +323,5 @@
         <origin xyz="0 0 0" rpy="0 0 0" />
         <inertia ixx="0.3" ixy="0.0" ixz="0.0" iyy="0.3" iyz="0.0" izz="0.3" />
-        <mass value="3.06" />
+        <mass value="0.45606" />
       </inertial>
     </link>
@@ -357,5 +357,5 @@
         <origin xyz="0 0 0" rpy="0 0 0" />
         <inertia ixx="0.3" ixy="0.0" ixz="0.0" iyy="0.3" iyz="0.0" izz="0.3" />
-        <mass value="3.06" />
+        <mass value="0.001" />
       </inertial>
     </link>
