Commit message: wall

File: robots/panda_arm.xacro (robot description, xacro)
@@ -6,4 +6,23 @@
     <xacro:property name="joint_damping" value="1.0"/>
     <link name="world" />
+    <link name="wall">
+      <visual>
+        <origin xyz="-0.1 0 1.5" rpy="0 0 0"/>
+        <geometry>
+          <box size="0.2 1 3" />
+        </geometry>
+      </visual>
+      <collision>
+        <origin xyz="-0.1 0 1.5" rpy="0 0 0"/>
+        <geometry>
+          <box size="0.2 1 3" />
+        </geometry>
+      </collision>
+    </link>
+    <joint name="dummy_joint" type="fixed">
+      <origin xyz="0 0 0" rpy="0 0 0" />
+      <parent link="world" />
+      <child link="wall" />
+    </joint>
     <xacro:unless value="${not connected_to}">
       <joint name="${arm_id}_joint_${connected_to}" type="fixed">
@@ -11,5 +30,4 @@
         <child link="${arm_id}_link0"/>
         <origin rpy="${rpy}" xyz="${xyz}"/>
-        <dynamics damping="${joint_damping}"/>
       </joint>
     </xacro:unless>

File: robots/panda_arm_hand.urdf.xacro (robot description, xacro)
@@ -3,5 +3,5 @@
   <xacro:include filename="$(find franka_description)/robots/panda_arm.xacro"/>
   <!-- <xacro:include filename="$(find franka_description)/robots/hand.xacro"/> -->
-  <xacro:panda_arm arm_id="panda" xyz="0 0 0" safety_distance="0.03" connected_to="world"/>
+  <xacro:panda_arm arm_id="panda" xyz="0 0 1.5" rpy="0 1.5708 0" safety_distance="0" connected_to="wall"/>
   <!-- <xacro:hand ns="panda" connected_to="panda_link8" /> -->
 </robot>

Commit message: Inertia

File: robots/panda_arm.xacro (robot description, xacro)
@@ -2,8 +2,27 @@
 <robot xmlns:xacro="http://www.ros.org/wiki/xacro" name="panda">
   <!-- safety_distance: Minimum safety distance in [m] by which the collision volumes are expanded and which is enforced during robot motions -->
-  <!-- arm_id: Namespace of the panda arm. Serves to differentiate between arms in case of multiple instances. -->
+  <!-- arm_id: Namespace of the paree.nda arm. Serves to differentiate between arms in case of multiple instances. -->
   <xacro:macro name="panda_arm" params="arm_id:='panda' description_pkg:='franka_description' connected_to:='' xyz:='0 0 0' rpy:='0 0 0' safety_distance:=0">
     <xacro:property name="joint_damping" value="1.0"/>
     <link name="world" />
+    <link name="wall">
+      <visual>
+        <origin xyz="-0.1 0 1.5" rpy="0 0 0"/>
+        <geometry>
+          <box size="0.2 1 3"/>
+        </geometry>
+      </visual>
+      <collision>
+        <origin xyz="-0.1 0 1.5" rpy="0 0 0"/>
+        <geometry>
+          <box size="0.2 1 3"/>
+        </geometry>
+      </collision>
+    </link>
+    <joint name="dummy_joint" type="fixed">
+      <parent link="world" />
+      <child link="wall" />
+      <origin xyz="0.0 0.0 0.0" rpy="0.0 0.0 0.0" />
+    </joint>
     <xacro:unless value="${not connected_to}">
       <joint name="${arm_id}_joint_${connected_to}" type="fixed">
@@ -11,5 +30,4 @@
         <child link="${arm_id}_link0"/>
         <origin rpy="${rpy}" xyz="${xyz}"/>
-        <dynamics damping="${joint_damping}"/>
       </joint>
     </xacro:unless>
@@ -69,7 +87,7 @@
       </collision>
       <inertial>
-        <origin xyz="0 0 0" rpy="0 0 0" />
-        <inertia ixx="0.3" ixy="0.0" ixz="0.0" iyy="0.3" iyz="0.0" izz="0.3" />
-        <mass value="2.34471" />
+        <origin xyz="0.0039 0.0021 0" rpy="0 0 0" />
+        <inertia ixx="0.703" ixy="-0.000139" ixz="0.00677" iyy="0.707" iyz="0.0192" izz="0.00912" />
+        <mass value="4.97" />
       </inertial>
     </link>
@@ -108,7 +126,7 @@
       </collision>
       <inertial>
-        <origin xyz="0 0 0" rpy="0 0 0" />
-        <inertia ixx="0.3" ixy="0.0" ixz="0.0" iyy="0.3" iyz="0.0" izz="0.3" />
-        <mass value="2.36414" />
+        <origin xyz="-0.00314 -0.0287 0.0035" rpy="0 0 0" />
+        <inertia ixx="0.00796" ixy="-0.00393" ixz="0.0103" iyy="0.0281" iyz="0.0007" izz="0.026" />
+        <mass value="0.647" />
       </inertial>
     </link>
@@ -147,7 +165,7 @@
       </collision>
       <inertial>
-        <origin xyz="0 0 0" rpy="0 0 0" />
-        <inertia ixx="0.3" ixy="0.0" ixz="0.0" iyy="0.3" iyz="0.0" izz="0.3" />
-        <mass value="2.38050" />
+        <origin xyz="0.0275 0.0393 -0.0665" rpy="0 0 0" />
+        <inertia ixx="0.0372" ixy="-0.00476" ixz="-0.0114" iyy="0.0362" iyz="-0.0128" izz="0.01083" />
+        <mass value="3.23" />
       </inertial>
     </link>
@@ -186,7 +204,7 @@
       </collision>
       <inertial>
-        <origin xyz="0 0 0" rpy="0 0 0" />
-        <inertia ixx="0.3" ixy="0.0" ixz="0.0" iyy="0.3" iyz="0.0" izz="0.3" />
-        <mass value="2.42754" />
+        <origin xyz="-0.0532 0.1044 0.0275" rpy="0 0 0" />
+        <inertia ixx="0.0259" ixy="0.0078" ixz="0.00133" iyy="0.01955" iyz="0.00864" izz="0.0283" />
+        <mass value="3.59" />
       </inertial>
     </link>
@@ -243,7 +261,7 @@
       </collision>
       <inertial>
-        <origin xyz="0 0 0" rpy="0 0 0" />
-        <inertia ixx="0.3" ixy="0.0" ixz="0.0" iyy="0.3" iyz="0.0" izz="0.3" />
-        <mass value="3.49611" />
+        <origin xyz="-0.012 0.0411 -0.0384" rpy="0 0 0" />
+        <inertia ixx="0.0355" ixy="-0.00212" ixz="-0.004037" iyy="0.0295" iyz="0.000229" izz="0.00863" />
+        <mass value="1.23" />
       </inertial>
     </link>
@@ -282,7 +300,7 @@
       </collision>
       <inertial>
-        <origin xyz="0 0 0" rpy="0 0 0" />
-        <inertia ixx="0.3" ixy="0.0" ixz="0.0" iyy="0.3" iyz="0.0" izz="0.3" />
-        <mass value="1.46736" />
+        <origin xyz="0.0602 -0.01412 -0.01052" rpy="0 0 0" />
+        <inertia ixx="0.001964" ixy="0.000109" ixz="-0.001158" iyy="0.00435" iyz="0.000341" izz="0.00543" />
+        <mass value="1.67" />
       </inertial>
     </link>
@@ -321,7 +339,7 @@
       </collision>
       <inertial>
-        <origin xyz="0 0 0" rpy="0 0 0" />
-        <inertia ixx="0.3" ixy="0.0" ixz="0.0" iyy="0.3" iyz="0.0" izz="0.3" />
-        <mass value="0.45606" />
+        <origin xyz="0.01052 -0.00425 0.0616" rpy="0 0 0" />
+        <inertia ixx="0.01252" ixy="-0.000428" ixz="-0.001196" iyy="0.01003" iyz="-0.000741" izz="0.00482" />
+        <mass value="0.736" />
       </inertial>
     </link>

File: robots/panda_arm_hand.urdf.xacro (robot description, xacro)
@@ -3,5 +3,5 @@
   <xacro:include filename="$(find franka_description)/robots/panda_arm.xacro"/>
   <!-- <xacro:include filename="$(find franka_description)/robots/hand.xacro"/> -->
-  <xacro:panda_arm arm_id="panda" xyz="0 0 0" safety_distance="0.03" connected_to="world"/>
+  <xacro:panda_arm arm_id="panda" xyz="0 0 1.5" rpy="0 1.5708 0" safety_distance="0" connected_to="wall"/>
   <!-- <xacro:hand ns="panda" connected_to="panda_link8" /> -->
 </robot>
